File: Orientation.kicad_sch (KiCad schematic)
At the start: 12 parts, among them J1 DIN41612_02x05_AB_EvenPins, J10 DIN41612_02x05_AB_EvenPins, J11 DIN41612_02x05_AB_EvenPins, J12 DIN41612_02x05_AB_EvenPins, J2 DIN41612_02x05_AB_EvenPins, J3 DIN41612_02x05_AB_EvenPins, J4 DIN41612_02x05_AB_EvenPins, J5 DIN41612_02x05_AB_EvenPins, J6 DIN41612_02x05_AB_EvenPins, J7 DIN41612_02x05_AB_EvenPins, J8 DIN41612_02x05_AB_EvenPins, J9 DIN41612_02x05_AB_EvenPins

Commit message: clarifying labels
Other:
- note added: "(+90 X)"
- note added: "(-90 X)"
- note added: "(0 X)"
- note added: "(0 Y)"
Changed lines of the file:
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@@
     (stroke (width 0) (type default) (color 0 0 0 0))
+  )
+  (text "(+90 X)" (at 106.68 68.58 0)
+    (effects (font (size 1.27 1.27)) (justify left bottom))
   )
   (text "Mirroring" (at 181.61 17.78 0)
@@
     (effects (font (size 1.27 1.27)) (justify left bottom))
   )
+  (text "(+90 X)" (at 203.2 64.77 0)
+    (effects (font (size 1.27 1.27)) (justify left bottom))
+  )
+  (text "(0 X)" (at 205.74 82.55 0)
+    (effects (font (size 1.27 1.27)) (justify left bottom))
+  )
   (text "+90º" (at 46.99 55.88 0)
     (effects (font (size 1.27 1.27)) (justify left bottom))
@@
     (effects (font (size 1.27 1.27)) (justify left bottom))
   )
+  (text "(-90 X)" (at 106.68 52.07 0)
+    (effects (font (size 1.27 1.27)) (justify left bottom))
+  )
   (text "Mirror X" (at 83.82 26.67 0)
     (effects (font (size 1.27 1.27)) (justify left bottom))
@@
     (effects (font (size 1.27 1.27)) (justify left bottom))
   )
+  (text "(0 Y)" (at 85.09 91.44 0)
+    (effects (font (size 1.27 1.27)) (justify left bottom))
+  )
+  (text "(0 Y)" (at 181.61 99.06 0)
+    (effects (font (size 1.27 1.27)) (justify left bottom))
+  )
   (text "0º" (at 147.32 38.1 0)
     (effects (font (size 1.27 1.27)) (justify left bottom))
   )
+  (text "(0 X)" (at 106.68 85.09 0)
+    (effects (font (size 1.27 1.27)) (justify left bottom))
+  )
+  (text "(-90 X)" (at 203.2 62.23 0)
+    (effects (font (size 1.27 1.27)) (justify left bottom))
+  )

Commit message: add new symbol
Parts:
- added U1, U10, U11, U12, U2, U3, U4, U5, U6, U7, U8, U9: Test1, symbol OrientationLib:Test1

Commit message: another symbol to test
Parts:
- added U? (x12): Test2, symbol OrientationLib:Test2
